File: dsPIC33CK256MC506_DevBoard.kicad_pcb (KiCad board)
At the start: 2 copper layers, 50.8 x 50.8 mm, 31 parts, among them J1 ICSP, J2 Pins_01_to_16, J3 Conn_02x06_Odd_Even, J4 Conn_01x02, J5 Conn_02x02_Odd_Even, J6 Pins_01_to_16, J7 Pins_17_to_32, Q1 DTC143Z, Q2 DTC143Z, Q3 DTC143Z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

Commit message: Updated documentation and component values
 - Schematic for analyzing
 - Schematic for printing
 - Interactive BOM for assembly
 - Updated component values
Parts:
- D1: value HB -> RED
- D2, D3, D4: value HB -> AMBAR
- R2, R3, R4, R5: value 470 -> 150
- Y1: value 10MHz@12ppm -> 10MHz@15ppm
